Commit message: add b2 urdf

File: urdf/b2.urdf (robot description, URDF)
Before this commit: robot B2, 1 links, 0 joints
Links:
- added link camera_link; visual box size=0.025 0.085 0.025
- link base_link: geometry visual box size=0.250 0.200 0.080; visual cylinder length=0.025 radius=0.0325
Joints:
- added joint camera_link_joint: type fixed, parent base_link, child camera_link, origin xyz=0.085 0.0 0.175 rpy=0.0 0.0 0.0

Commit message: add imu_link, fix base_link origins

File: urdf/b2.urdf (robot description, URDF)
Before this commit: robot B2, 2 links, 1 joints
Links:
- added link imu_link; visual box size=0.02032 0.0127 0.003
- link base_link: geometry visual box size=0.250 0.200 0.075; visual cylinder length=0.025 radius=0.0325
Joints:
- added joint imu_link_join: type fixed, parent base_link, child imu_link, origin xyz=-0.070 -0.040 0.135 rpy=0.0 0.0 0.0
- joint camera_link_joint: origin xyz=0.085 0.0 0.175 rpy=0.0 0.0 0.0 -> xyz=0.085 0.0 0.238 rpy=0.0 0.0 0.0

Commit message: adjust for NUC8 mounting

File: urdf/b2.urdf (robot description, URDF)
Before this commit: robot B2, 3 links, 2 joints
Links:
- link base_link: geometry visual box size=0.055 0.085 0.010; visual box size=0.070 0.095 0.030
Joints:
- joint camera_link_joint: origin xyz=0.085 0.0 0.238 rpy=0.0 0.0 0.0 -> xyz=0.118 0.0 0.214 rpy=0.0 0.0 0.0
- joint imu_link_join: origin xyz=-0.070 -0.040 0.135 rpy=0.0 0.0 0.0 -> xyz=-0.070 -0.016 0.1675 rpy=0.0 0.0 0.0

Commit message: rearrange for adding rplidar and sensor arch

File: urdf/b2.urdf (robot description, URDF)
Before this commit: robot B2, 3 links, 2 joints
Links:
- added link scanner_link; visual box size=0.100 0.070 0.033; visual cylinder length=0.024 radius=0.035
- link base_link: geometry visual box size=0.035 0.045 0.010; visual box size=0.070 0.094 0.030
Joints:
- added joint scanner_link_join: type fixed, parent base_link, child scanner_link, origin xyz=0.080 0 0.228 rpy=0.0 0.0 3.14159
- joint camera_link_joint: origin xyz=0.118 0.0 0.214 rpy=0.0 0.0 0.0 -> xyz=0.143 0.0 0.185 rpy=0.0 0.0 0.0
- joint imu_link_join: origin xyz=-0.070 -0.016 0.1675 rpy=0.0 0.0 0.0 -> xyz=0.080 -0.035 0.133 rpy=0.0 0.0 0.0

Commit message: add initial xacro

File: urdf/b2.urdf (robot description, URDF)
Before this commit: robot B2, 4 links, 3 joints
Links:
- link base_link: geometry visual box size=${base_x_len} ${base_y_width} ${base_box_ht}; visual box size=0.070 0.094 0.030
Joints:
- joint imu_link_join: origin xyz=0.080 -0.035 0.133 rpy=0.0 0.0 0.0 -> xyz=0.040 -0.040 ${base_box_top_ht + sensor_arch_ht + 0.008} rpy=0.0 0.0 0.0
